File: telemach-mp157-dev-board-shield.kicad_pcb (KiCad board)
At the start: 4 copper layers, 120 x 66 mm, 5 parts, among them CON1 2x17x2.54mm, CON10 77313-818-08LF, CON11 1x2x2.54mm, CON2 1x9x2.54mm, CON8 2x17x2.54mm

Commit message: Template is ready
Parts:
- removed CON10: 77313-818-08LF, Goldpin:Goldpin_4_2_2_54mm
- removed CON11: 1x2x2.54mm, Goldpin:Goldpin_2_2_54mm
- removed CON8: 2x17x2.54mm, Goldpin:Goldpin_17_2_2_54mm_SMT
- added CON3: Header_Socket_1x9pin, Header_Socket_2_54mm:Header_Socket_1x9x2_54mm, B.Cu at (178.8, 81.5)
- added CON4: Header_Socket_2x4pin, Header_Socket_2_54mm:Header_Socket_2x4x2_54mm, B.Cu at (208.1, 130.4)
- added CON5: Header_Socket_1x2pin, Header_Socket_2_54mm:Header_Socket_1x2x2_54mm, B.Cu at (161.7, 81.5)
- CON1: value 2x17x2.54mm -> Header_Socket_2x17pin; footprint Goldpin:Goldpin_17_2_2_54mm_SMT -> Header_Socket_2_54mm:Header_Socket_2x17x2_54mm; moved to B.Cu
- CON2: value 1x9x2.54mm -> Header_Socket_2x17pin; footprint Goldpin:Goldpin_9_2_54mm -> Header_Socket_2_54mm:Header_Socket_2x17x2_54mm; moved to B.Cu
- moved CON2 49.9 mm to (162.1, 128.5), turned to 180 degrees
- turned CON1 to 180 degrees
Connections:
- CON1 pad 1: /Gold Connector/PIN1 -> unconnected-(CON1-Pad1)
- CON1 pad 10: /Gold Connector/PIN10 -> unconnected-(CON1-Pad10)
- CON1 pad 11: /Gold Connector/PIN11 -> unconnected-(CON1-Pad11)
- CON1 pad 12: /Gold Connector/PIN12 -> unconnected-(CON1-Pad12)
- CON1 pad 13: /Gold Connector/PIN13 -> unconnected-(CON1-Pad13)
- CON1 pad 14: /Gold Connector/PIN14 -> unconnected-(CON1-Pad14)
- CON1 pad 15: /Gold Connector/PIN15 -> unconnected-(CON1-Pad15)
- CON1 pad 16: /Gold Connector/PIN16 -> unconnected-(CON1-Pad16)
- CON1 pad 17: /Gold Connector/PIN17 -> unconnected-(CON1-Pad17)
- CON1 pad 18: /Gold Connector/PIN18 -> unconnected-(CON1-Pad18)
- CON1 pad 19: /Gold Connector/PIN19 -> unconnected-(CON1-Pad19)
- CON1 pad 2: GND -> unconnected-(CON1-Pad2)
- CON1 pad 20: /Gold Connector/PIN20 -> unconnected-(CON1-Pad20)
- CON1 pad 21: /Gold Connector/PIN21 -> unconnected-(CON1-Pad21)
- CON1 pad 22: /Gold Connector/PIN22 -> unconnected-(CON1-Pad22)
- CON1 pad 23: /Gold Connector/PIN23 -> unconnected-(CON1-Pad23)
- CON1 pad 24: /Gold Connector/PIN24 -> unconnected-(CON1-Pad24)
- CON1 pad 25: /Gold Connector/PIN25 -> unconnected-(CON1-Pad25)
- CON1 pad 26: /Gold Connector/PIN26 -> unconnected-(CON1-Pad26)
- CON1 pad 27: /Gold Connector/PIN27 -> unconnected-(CON1-Pad27)
- CON1 pad 28: /Gold Connector/PIN28 -> unconnected-(CON1-Pad28)
- CON1 pad 29: /Gold Connector/PIN29 -> unconnected-(CON1-Pad29)
- CON1 pad 3: 5V -> unconnected-(CON1-Pad3)
- CON1 pad 30: /Gold Connector/PIN30 -> unconnected-(CON1-Pad30)
- CON1 pad 31: /Gold Connector/PIN31 -> unconnected-(CON1-Pad31)
- CON1 pad 32: /Gold Connector/PIN32 -> unconnected-(CON1-Pad32)
- CON1 pad 33: /Gold Connector/PIN33 -> unconnected-(CON1-Pad33)
- CON1 pad 34: /Gold Connector/PIN34 -> unconnected-(CON1-Pad34)
- CON1 pad 4: /Gold Connector/PIN4 -> unconnected-(CON1-Pad4)
- CON1 pad 5: /Gold Connector/PIN5 -> unconnected-(CON1-Pad5)
- CON1 pad 6: /Gold Connector/PIN6 -> unconnected-(CON1-Pad6)
- CON1 pad 7: /Gold Connector/PIN7 -> unconnected-(CON1-Pad7)
- CON1 pad 8: /Gold Connector/PIN8 -> unconnected-(CON1-Pad8)
- CON1 pad 9: /Gold Connector/PIN9 -> unconnected-(CON1-Pad9)
- CON2 pad 1: GND -> unconnected-(CON2-Pad1)
- CON2 pad 2: GND -> unconnected-(CON2-Pad2)
- CON2 pad 3: 3V3 -> unconnected-(CON2-Pad3)
- CON2 pad 4: 3V3 -> unconnected-(CON2-Pad4)
- CON2 pad 5: /MCU Unit/PD1_GPIO -> unconnected-(CON2-Pad5)
- CON2 pad 6: /MCU Unit/PB7_GPIO -> unconnected-(CON2-Pad6)
- CON2 pad 7: /MCU Unit/JTCK-SWCLK -> unconnected-(CON2-Pad7)
- CON2 pad 8: /MCU Unit/PD5_GPIO -> unconnected-(CON2-Pad8)
- CON2 pad 9: /MCU Unit/JTMS-SWDIO -> unconnected-(CON2-Pad9)
Other:
- board text added: "PONKEY"
- board text removed: "PNKEY"
