File: telemach-mp157-dev-board-shield.kicad_sch (KiCad schematic)
At the start: 0 parts

Commit message: Template is ready
Parts:
- added CON1, CON2: Header_Socket_2x17pin, Header_Socket_2_54mm:Header_Socket_2x17x2_54mm, symbol Header_Socket_2_54mm:Header_Socket_2x17pin
- added CON3: Header_Socket_1x9pin, Header_Socket_2_54mm:Header_Socket_1x9x2_54mm, symbol Header_Socket_2_54mm:Header_Socket_1x9pin
- added CON4: Header_Socket_2x4pin, Header_Socket_2_54mm:Header_Socket_2x4x2_54mm, symbol Header_Socket_2_54mm:Header_Socket_2x4pin
- added CON5: Header_Socket_1x2pin, Header_Socket_2_54mm:Header_Socket_1x2x2_54mm, symbol Header_Socket_2_54mm:Header_Socket_1x2pin
